File: cad/pcb/spc_evdr.kicad_pcb (KiCad board)
At the start: 2 copper layers, 197 x 97.5 mm, 91 parts, among them J1 BL_CONN, SW1 SW_Push, SW10 SW_Push, SW11 SW_Push, SW12 SW_Push, SW13 ON_OFF, SW14 SW_Push, SW15 SW_Push, SW16 SW_Push, SW17 SW_Push, SW18 SW_Push, SW19 SW_Push, SW2 SW_Push, SW20 SW_Push, SW21 SW_Push, SW22 SW_Push, SW23 SW_Push, SW24 SW_Push, SW25 SW_Push, SW26 SW_Push, SW27 SW_Push, SW28 SW_Push, SW29 SW_Push, SW3 SW_Push, SW30 SW_Push, SW31 SW_Push, SW32 SW_Push, SW33 SW_Push, SW34 SW_Push, SW35 SW_Push, SW36 SW_Push, SW37 SW_Push, SW38 SW_Push, SW39 SW_Push, SW4 SW_Push, SW40 SW_Push, SW41 SW_Push, SW42 SW_Push, SW43 SW_Push, SW44 SW_Push, SW45 SW_Push, SW6 SW_Push, SW7 SW_Push, SW8 SW_Push, SW9 SW_Push, U1 PCA9555PW, U2 xiao-ble

Commit message: update pcb files
Parts:
- added D39: D_Small, weteor:D_SOD-123, B.Cu at (109.2, 23.6)
- added SW5: RotaryEncoder_Switch, weteor:ec11_smd, F.Cu at (54.7, 18.6)
- BT1: moved to B.Cu
- SW1, SW10, SW11, SW12, SW14, SW15, SW16, SW17, SW2, SW20, SW21, SW22, SW25, SW26, SW27, SW3, SW31, SW32, SW33, SW34, SW35, SW36, SW37, SW38, SW39, SW4, SW40, SW41, SW42, SW43, SW44, SW45, SW6, SW7, SW8, SW9: footprint weteor:CherryMX_Hotswap -> weteor:Inv1_CherryMX_Hotswap
- SW18, SW29: footprint weteor:CherryMX_Hotswap_1.25u -> weteor:Inv_CherryMX_Hotswap_1.25u
- SW19, SW30: footprint weteor:CherryMX_Hotswap_2.25u_stabs -> weteor:InvCherryMX_Hotswap_2.25u_stabs
- SW23, SW28: footprint weteor:CherryMX_Hotswap_1.75u -> weteor:Inv_CherryMX_Hotswap_1.75u
- SW24: footprint weteor:CherryMX_Hotswap_3u_stabs -> weteor:InvCherryMX_Hotswap_3u_stabs
- moved SW13 57.1 mm to (122.6, 17.9)
- moved D15 17.9 mm to (132.2, 109.5)
- moved D27 17.9 mm to (153.6, 109.5)
- moved D24 8.33 mm to (179.8, 47.6)
- moved D25 8.33 mm to (179.8, 66.7)
- moved D26 8.33 mm to (179.8, 85.7)
- moved D6 8.33 mm to (67.9, 47.6)
- moved D7 8.33 mm to (67.9, 66.7)
- moved D8 8.33 mm to (67.9, 85.7)
- moved D1 8.33 mm to (65.5, 47.6)
- moved D2 8.33 mm to (65.5, 66.7)
- moved D3 8.33 mm to (65.5, 85.7)
- moved D10 8.33 mm to (103.6, 66.7)
- moved D11 8.33 mm to (103.6, 85.7)
- moved D12 8.33 mm to (106.0, 47.6)
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Connections:
- U2 pad 1: unconnected-(U2-Pad1) -> encA
- U2 pad 2: unconnected-(U2-Pad2) -> encB
Routing:
- net encB: track 0.00 -> 211.4 mm, vias 0 -> 3
- net encA: track 0.00 -> 208.4 mm, vias 0 -> 3
- net Col_3: track 82.3 -> 165.4 mm, vias 4 -> 6
- net Net-(D39-Pad2): track 0.00 -> 63.5 mm, vias 0 -> 1
- net Net-(BT1-Pad1): track 67.7 -> 7.18 mm, vias 2 -> 1
- net Row_1: track 251.6 -> 221.9 mm
- net Row_4: track 274.9 -> 292.9 mm, vias 2 -> 3
- net Net-(D27-Pad2): track 10.3 -> 28.2 mm
- net Row_3: track 239.9 -> 223.2 mm
- net Row_2: track 217.4 -> 200.8 mm
- net Net-(D15-Pad2): track 72.5 -> 88.5 mm
- net Net-(SW13-Pad2): track 51.0 -> 36.7 mm, vias 1 -> 3
- net Net-(D2-Pad2): track 8.25 -> 16.8 mm
- net Net-(D17-Pad2): track 8.25 -> 16.8 mm
- net Net-(D33-Pad2): track 8.25 -> 16.7 mm
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Other:
- board size 197 x 97.5 mm -> 199.5 x 100.5 mm
