File: cad/pcb/spc_evdr.kicad_sch (KiCad schematic)
At the start: 91 parts, among them J1 BL_CONN, SW1 SW_Push, SW10 SW_Push, SW11 SW_Push, SW12 SW_Push, SW13 ON_OFF, SW14 SW_Push, SW15 SW_Push, SW16 SW_Push, SW17 SW_Push, SW18 SW_Push, SW19 SW_Push, SW2 SW_Push, SW20 SW_Push, SW21 SW_Push, SW22 SW_Push, SW23 SW_Push, SW24 SW_Push, SW25 SW_Push, SW26 SW_Push, SW27 SW_Push, SW28 SW_Push, SW29 SW_Push, SW3 SW_Push, SW30 SW_Push, SW31 SW_Push, SW32 SW_Push, SW33 SW_Push, SW34 SW_Push, SW35 SW_Push, SW36 SW_Push, SW37 SW_Push, SW38 SW_Push, SW39 SW_Push, SW4 SW_Push, SW40 SW_Push, SW41 SW_Push, SW42 SW_Push, SW43 SW_Push, SW44 SW_Push, SW45 SW_Push, SW6 SW_Push, SW7 SW_Push, SW8 SW_Push, SW9 SW_Push, U1 PCA9555PW, U2 xiao-ble

Commit message: update pcb files
Parts:
- added D39: D_Small, Diode_SMD:D_SOD-123, symbol Device:D_Small
- added SW5: RotaryEncoder_Switch, Rotary_Encoder:RotaryEncoder_Alps_EC11E-Switch_Vertical_H20mm, symbol Device:RotaryEncoder_Switch
Connections:
- net Col_3: now also SW5.S1
- net GND: now also SW5.C
- net Row_4: now also D39.1 (K)
- net encA: now reaches U2.1 (A2/0.02_H)
- net encA: now also SW5.A
- net encB: now reaches U2.2 (A4/0.03_H)
- net encB: now also SW5.B
- new net: D39.2 (A), SW5.S2
- no-connect marks 15 -> 13
Changed lines of the file:
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@@
   )
   (no_connect (at 158.75 140.335))
-  (no_connect (at 115.57 140.335))
   (no_connect (at 69.85 158.75))
   (no_connect (at 69.85 161.29))
@@
   (no_connect (at 135.89 164.465))
   (no_connect (at 138.43 164.465))
-  (no_connect (at 115.57 142.875))
   (no_connect (at 115.57 145.415))
   (wire (pts (xy 240.665 139.065) (xy 241.3 139.065))
@@
     (stroke (width 0) (type default) (color 0 0 0 0))
   )
+  (wire (pts (xy 45.085 94.615) (xy 48.895 94.615))
+    (stroke (width 0) (type default) (color 0 0 0 0))
+  )
   (wire (pts (xy 238.76 50.8) (xy 241.3 50.8))
     (stroke (width 0) (type default) (color 0 0 0 0))
@@
     (stroke (width 0) (type default) (color 0 0 0 0))
   )
+  (wire (pts (xy 22.225 97.155) (xy 29.845 97.155))
+    (stroke (width 0) (type default) (color 0 0 0 0))
+  )
   (wire (pts (xy 116.205 170.18) (xy 130.81 170.18))
     (stroke (width 0) (type default) (color 0 0 0 0))
@@
     (stroke (width 0) (type default) (color 0 0 0 0))
   )
+  (wire (pts (xy 110.49 142.875) (xy 115.57 142.875))
+    (stroke (width 0) (type default) (color 0 0 0 0))
+  )
   (wire (pts (xy 133.35 19.05) (xy 133.35 25.4))
     (stroke (width 0) (type default) (color 0 0 0 0))
@@
     (stroke (width 0) (type default) (color 0 0 0 0))
   )
+  (wire (pts (xy 47.625 104.775) (xy 47.625 107.315))
+    (stroke (width 0) (type default) (color 0 0 0 0))
+  )
   (wire (pts (xy 209.55 38.1) (xy 209.55 50.8))
     (stroke (width 0) (type default) (color 0 0 0 0))
@@
     (stroke (width 0) (type default) (color 0 0 0 0))
   )
+  (wire (pts (xy 45.085 99.695) (xy 47.625 99.695))
+    (stroke (width 0) (type default) (color 0 0 0 0))
+  )
   (wire (pts (xy 53.975 25.4) (xy 53.975 38.1))
     (stroke (width 0) (type default) (color 0 0 0 0))
@@
     (stroke (width 0) (type default) (color 0 0 0 0))
   )
+  (wire (pts (xy 110.49 140.335) (xy 115.57 140.335))
+    (stroke (width 0) (type default) (color 0 0 0 0))
+  )
   (wire (pts (xy 69.85 30.48) (xy 88.9 30.48))
     (stroke (width 0) (type default) (color 0 0 0 0))
@@
   )
   (wire (pts (xy 74.295 153.67) (xy 69.85 153.67))
+    (stroke (width 0) (type default) (color 0 0 0 0))
+  )
+  (wire (pts (xy 47.625 107.315) (xy 49.53 107.315))
     (stroke (width 0) (type default) (color 0 0 0 0))
   )
@@
     )
   )
+  (global_label "encB" (shape input) (at 110.49 142.875 180)
+    (effects (font (size 1.27 1.27)) (justify right))
+    (property "Intersheetrefs" "${INTERSHEET_REFS}" (id 0) (at -133.35 60.325 0)
+      (effects (font (size 1.27 1.27)) hide)
+    )
+  )
   (global_label "Row_1" (shape input) (at 247.65 30.48 0) (fields_autoplaced)
     (effects (font (size 1.27 1.27)) (justify left))
@@
     (effects (font (size 1.27 1.27)) (justify left))
     (property "Intersheet References" "${INTERSHEET_REFS}" (id 0) (at 53.8956 11.3755 90)
+      (effects (font (size 1.27 1.27)) (justify left) hide)
+    )
+  )
+  (global_label "Row_4" (shape input) (at 49.53 107.315 0) (fields_autoplaced)
+    (effects (font (size 1.27 1.27)) (justify left))
+    (property "Intersheet References" "${INTERSHEET_REFS}" (id 0) (at 57.8698 107.2356 0)
       (effects (font (size 1.27 1.27)) (justify left) hide)
     )
@@
     )
   )
+  (global_label "encB" (shape input) (at 29.845 99.695 180)
+    (effects (font (size 1.27 1.27)) (justify right))
+    (property "Intersheetrefs" "${INTERSHEET_REFS}" (id 0) (at -213.995 17.145 0)
+      (effects (font (size 1.27 1.27)) hide)
+    )
+  )
   (global_label "Row_2" (shape input) (at 247.65 43.18 0) (fields_autoplaced)
     (effects (font (size 1.27 1.27)) (justify left))
@@
     (property "Intersheet References" "${INTERSHEET_REFS}" (id 0) (at 114.2206 11.3755 90)
       (effects (font (size 1.27 1.27)) (justify left) hide)
+    )
+  )
+  (global_label "encA" (shape input) (at 29.845 94.615 180)
+    (effects (font (size 1.27 1.27)) (justify right))
+    (property "Intersheetrefs" "${INTERSHEET_REFS}" (id 0) (at -213.995 17.145 0)
+      (effects (font (size 1.27 1.27)) hide)
     )
   )
@@
     )
   )
+  (global_label "encA" (shape input) (at 110.49 140.335 180)
+    (effects (font (size 1.27 1.27)) (justify right))
+    (property "Intersheetrefs" "${INTERSHEET_REFS}" (id 0) (at -133.35 62.865 0)
+      (effects (font (size 1.27 1.27)) hide)
+    )
+  )
   (global_label "sda" (shape input) (at 231.775 139.065 180)
     (effects (font (size 1.27 1.27)) (justify right))
@@
     (effects (font (size 1.27 1.27)) (justify left))
     (property "Intersheet References" "${INTERSHEET_REFS}" (id 0) (at 209.4706 11.3755 90)
+      (effects (font (size 1.27 1.27)) (justify left) hide)
+    )
+  )
+  (global_label "Col_3" (shape input) (at 48.895 94.615 0) (fields_autoplaced)
+    (effects (font (size 1.27 1.27)) (justify left))
+    (property "Intersheet References" "${INTERSHEET_REFS}" (id 0) (at 56.5695 94.5356 0)
       (effects (font (size 1.27 1.27)) (justify left) hide)
     )
@@
     (pin "2")
   )
+  (symbol (lib_id "power:GND") (at 22.225 97.155 0) (unit 1)
+    (in_bom yes) (on_board yes)
+    (property "Reference" "#PWR013" (id 0) (at 22.225 103.505 0)
+      (effects (font (size 1.27 1.27)) hide)
+    )
+    (property "Value" "GND" (id 1) (at 22.352 101.5492 0))
+    (property "Footprint" "" (id 2) (at 22.225 97.155 0)
+      (effects (font (size 1.27 1.27)) hide)
+    )
+    (property "Datasheet" "" (id 3) (at 22.225 97.155 0)
+      (effects (font (size 1.27 1.27)) hide)
+    )
+    (pin "1")
+  )
   (symbol (lib_id "Switch:SW_Push") (at 157.48 88.9 0) (unit 1)
     (in_bom yes) (on_board yes)
@@
     (pin "2")
   )
+  (symbol (lib_id "Device:D_Small") (at 47.625 102.235 90) (unit 1)
+    (in_bom yes) (on_board yes)
+    (property "Reference" "D39" (id 0) (at 49.403 101.0666 90)
+      (effects (font (size 1.27 1.27)) (justify right))
+    )
+    (property "Value" "D_Small" (id 1) (at 49.403 103.378 90)
+      (effects (font (size 1.27 1.27)) (justify right))
+    )
+    (property "Footprint" "Diode_SMD:D_SOD-123" (id 2) (at 47.625 102.235 90)
+      (effects (font (size 1.27 1.27)) hide)
+    )
+    (property "Datasheet" "~" (id 3) (at 47.625 102.235 90)
+      (effects (font (size 1.27 1.27)) hide)
+    )
+    (pin "1")
+    (pin "2")
+  )
   (symbol (lib_id "power:GND") (at 57.15 186.055 0) (unit 1)
     (in_bom yes) (on_board yes)
@@
     (pin "1")
     (pin "2")
+  )
+  (symbol (lib_id "Device:RotaryEncoder_Switch") (at 37.465 97.155 0) (unit 1)
+    (in_bom yes) (on_board yes) (fields_autoplaced)
+    (property "Reference" "SW5" (id 0) (at 37.465 88.3752 0))
+    (property "Value" "RotaryEncoder_Switch" (id 1) (at 37.465 90.9121 0))
+    (property "Footprint" "Rotary_Encoder:RotaryEncoder_Alps_EC11E-Switch_Vertical_H20mm" (id 2) (at 33.655 93.091 0)
+      (effects (font (size 1.27 1.27)) hide)
+    )
+    (property "Datasheet" "~" (id 3) (at 37.465 90.551 0)
+      (effects (font (size 1.27 1.27)) hide)
+    )
+    (pin "A")
+    (pin "B")
+    (pin "C")
+    (pin "S1")
+    (pin "S2")
   )
   (symbol (lib_id "Device:D_Small") (at 69.85 93.98 90) (unit 1)
@@
       (reference "#PWR012") (unit 1) (value "+3V3") (footprint "")
     )
+    (path "/2a690215-504e-4a44-ab6e-228c86d95cad"
+      (reference "#PWR013") (unit 1) (value "GND") (footprint "")
+    )
     (path "/1e915edd-3c71-4166-9103-db0e8b799037"
       (reference "BT1") (unit 1) (value "Battery_Cell") (footprint "Connector_Molex:Molex_PicoBlade_53048-0210_1x02_P1.25mm_Horizontal")
@@
       (reference "D38") (unit 1) (value "D") (footprint "weteor:D_SOD-123")
     )
+    (path "/30e6f2f1-03a3-43da-91bc-e44abf7ea547"
+      (reference "D39") (unit 1) (value "D_Small") (footprint "Diode_SMD:D_SOD-123")
+    )
     (path "/7b299874-7431-43f9-a847-bb61a7a1c4c9"
       (reference "J1") (unit 1) (value "BL_CONN") (footprint "Connector_PinHeader_2.54mm:PinHeader_1x04_P2.54mm_Vertical")
@@
       (reference "SW4") (unit 1) (value "SW_Push") (footprint "weteor:CherryMX_Hotswap")
     )
+    (path "/3eb0478a-75a7-4dc9-986e-b3e0235d47b7"
+      (reference "SW5") (unit 1) (value "RotaryEncoder_Switch") (footprint "Rotary_Encoder:RotaryEncoder_Alps_EC11E-Switch_Vertical_H20mm")
+    )
     (path "/05f1a344-8030-44b9-beaa-320b3e6a92cc"
